File: eagle/808-Diginoise.brd (EAGLE design)
At the start: 100 x 80 mm, 28 parts, among them IC1 4584N, IC2 TL071P, U1 POWER

Commit message: tweaks
Parts:
- moved R7 4.84 mm to (34.3, 69.2), turned to 90 degrees
Routing:
- net N$5: track 22.2 -> 13.4 mm
- net GND: track 206.4 -> 208.9 mm
- net N$18: track 91.8 -> 93.6 mm
Changed lines of the file:
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@@
 <element name="R5" library="TR808clone" package="0207/5V" value="100K" x="40.64" y="53.975" rot="R270"/>
 <element name="R6" library="TR808clone" package="0207/5V" value="150K" x="42.545" y="59.055" rot="R180"/>
-<element name="R7" library="TR808clone" package="0207/5V" value="120K" x="36.195" y="73.66" rot="R180"/>
+<element name="R7" library="TR808clone" package="0207/5V" value="120K" x="34.29" y="69.215" rot="R90"/>
 <element name="R8" library="TR808clone" package="0207/5V" value="120K" x="34.29" y="41.91" rot="R180"/>
 <element name="R9" library="TR808clone" package="0207/5V" value="120K" x="34.29" y="44.45" rot="R180"/>
@@
 <wire x1="32.385" y1="76.835" x2="16.8275" y2="76.835" width="1.016" layer="16"/>
 <wire x1="36.195" y1="74.93" x2="32.385" y2="76.835" width="1.016" layer="16"/>
-<wire x1="36.195" y1="72.39" x2="36.195" y2="74.93" width="1.016" layer="16"/>
-<wire x1="33.655" y1="71.755" x2="36.195" y2="72.39" width="1.016" layer="16"/>
-<wire x1="32.385" y1="70.485" x2="33.655" y2="71.755" width="1.016" layer="16"/>
-<wire x1="30.7975" y1="73.3425" x2="32.385" y2="70.485" width="1.016" layer="16"/>
+<wire x1="36.195" y1="69.215" x2="36.195" y2="74.93" width="1.016" layer="16"/>
+<wire x1="32.385" y1="69.215" x2="36.195" y2="69.215" width="1.016" layer="16"/>
+<wire x1="30.7975" y1="73.3425" x2="32.385" y2="69.215" width="1.016" layer="16"/>
 <wire x1="26.9875" y1="73.3425" x2="30.7975" y2="73.3425" width="1.016" layer="16"/>
 <wire x1="26.9875" y1="73.3425" x2="26.67" y2="73.66" width="1.016" layer="16"/>
@@
 <wire x1="46.0375" y1="41.5925" x2="43.815" y2="38.735" width="1.016" layer="16"/>
 <wire x1="46.0375" y1="41.5925" x2="46.45" y2="44.45" width="1.016" layer="16"/>
-<wire x1="32.385" y1="49.53" x2="32.385" y2="70.485" width="1.016" layer="16"/>
+<wire x1="32.385" y1="49.53" x2="32.385" y2="69.215" width="1.016" layer="16"/>
 <wire x1="29.5275" y1="47.9425" x2="32.385" y2="49.53" width="1.016" layer="16"/>
 <wire x1="29.5275" y1="47.9425" x2="29.21" y2="48.26" width="1.016" layer="16"/>
@@
 <contactref element="R6" pad="2"/>
 <wire x1="40.005" y1="59.055" x2="36.83" y2="58.42" width="0.8128" layer="16"/>
-<wire x1="38.1" y1="71.12" x2="38.735" y2="73.66" width="0.8128" layer="16"/>
-<wire x1="33.9725" y1="66.9925" x2="38.1" y2="71.12" width="0.8128" layer="16"/>
-<wire x1="33.9725" y1="59.69" x2="33.9725" y2="66.9925" width="0.8128" layer="16"/>
+<wire x1="33.9725" y1="65.7225" x2="34.29" y2="66.675" width="0.8128" layer="16"/>
+<wire x1="33.9725" y1="59.69" x2="33.9725" y2="65.7225" width="0.8128" layer="16"/>
 <wire x1="36.5125" y1="58.42" x2="33.9725" y2="59.69" width="0.8128" layer="16"/>
 <wire x1="36.5125" y1="58.42" x2="36.83" y2="58.42" width="0.8128" layer="16"/>
@@
 <wire x1="19.05" y1="71.4375" x2="21.59" y2="73.3425" width="0.8128" layer="16"/>
 <wire x1="19.05" y1="62.23" x2="19.05" y2="71.4375" width="0.8128" layer="16"/>
-<wire x1="31.4325" y1="75.2475" x2="33.655" y2="73.66" width="0.8128" layer="16"/>
+<wire x1="31.4325" y1="75.2475" x2="34.29" y2="71.755" width="0.8128" layer="16"/>
 <wire x1="23.495" y1="75.2475" x2="31.4325" y2="75.2475" width="0.8128" layer="16"/>
 <wire x1="21.9075" y1="73.66" x2="23.495" y2="75.2475" width="0.8128" layer="16"/>
