File: eagle/808-Diginoise.sch (EAGLE design)
At the start: 28 parts, among them IC1 4584N, IC2 TL071P, U1 POWER

Commit message: routed
Parts:
- renumbered JCK1 to OUTPUT, R2 to LEVEL
Changed lines of the file:
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@@
 <part name="P+1" library="supply1" deviceset="+12V" device=""/>
 <part name="P-2" library="supply1" deviceset="-12V" device=""/>
-<part name="JCK1" library="erthenvar" deviceset="AUDIO-JACK" device=""/>
+<part name="OUTPUT" library="erthenvar" deviceset="AUDIO-JACK" device=""/>
 <part name="GND10" library="supply1" deviceset="GND" device=""/>
 <part name="JP1" library="adafruit" deviceset="PINHD-2X4" device=""/>
 <part name="GND11" library="supply1" deviceset="GND" device=""/>
-<part name="R2" library="pot" deviceset="3RP/1610N" device="" value="100k"/>
+<part name="LEVEL" library="pot" deviceset="3RP/1610N" device="" value="100k"/>
 <part name="GND12" library="supply1" deviceset="GND" device=""/>
 </parts>
@@
 <instance part="P+1" gate="1" x="76.2" y="68.58"/>
 <instance part="P-2" gate="1" x="76.2" y="43.18"/>
-<instance part="JCK1" gate="G$1" x="121.92" y="45.72" rot="R180"/>
+<instance part="OUTPUT" gate="G$1" x="121.92" y="45.72" rot="R180"/>
 <instance part="GND10" gate="1" x="114.3" y="35.56"/>
 <instance part="JP1" gate="A" x="78.74" y="12.7"/>
 <instance part="GND11" gate="1" x="91.44" y="0"/>
-<instance part="R2" gate="G$1" x="93.98" y="50.8"/>
+<instance part="LEVEL" gate="G$1" x="93.98" y="50.8"/>
 <instance part="GND12" gate="1" x="93.98" y="35.56"/>
 </instances>
@@
 </segment>
 <segment>
-<pinref part="JCK1" gate="G$1" pin="RING"/>
+<pinref part="OUTPUT" gate="G$1" pin="RING"/>
 <pinref part="GND10" gate="1" pin="GND"/>
 <wire x1="114.3" y1="38.1" x2="114.3" y2="43.18" width="0.1524" layer="91"/>
@@
 </segment>
 <segment>
-<pinref part="R2" gate="G$1" pin="A"/>
+<pinref part="LEVEL" gate="G$1" pin="A"/>
 <pinref part="GND12" gate="1" pin="GND"/>
 <wire x1="93.98" y1="38.1" x2="93.98" y2="45.72" width="0.1524" layer="91"/>
@@
 <wire x1="68.58" y1="38.1" x2="88.9" y2="38.1" width="0.1524" layer="91"/>
 <wire x1="88.9" y1="38.1" x2="88.9" y2="55.88" width="0.1524" layer="91"/>
-<pinref part="R2" gate="G$1" pin="E"/>
+<pinref part="LEVEL" gate="G$1" pin="E"/>
 <wire x1="93.98" y1="55.88" x2="88.9" y2="55.88" width="0.1524" layer="91"/>
 <junction x="88.9" y="55.88"/>
@@
 <net name="N$7" class="0">
 <segment>
-<pinref part="R2" gate="G$1" pin="S"/>
+<pinref part="LEVEL" gate="G$1" pin="S"/>
 <pinref part="R1" gate="G$1" pin="2"/>
 <wire x1="101.6" y1="50.8" x2="99.06" y2="50.8" width="0.1524" layer="91"/>
@@
 <net name="N$16" class="0">
 <segment>
-<pinref part="JCK1" gate="G$1" pin="TIP"/>
+<pinref part="OUTPUT" gate="G$1" pin="TIP"/>
 <pinref part="R1" gate="G$1" pin="1"/>
 <wire x1="111.76" y1="50.8" x2="114.3" y2="50.8" width="0.1524" layer="91"/>
